File: adc.sch (EAGLE design)
At the start: 86 parts, among them IC13 4051D, IC5 4051D, IC6 4051D, U1 ADV7173KSTZ, U2 AD5308ARUZ, U3 AD7927BRUZ, U4 ADV7173KSTZ, U5 AD5308ARUZ, U6 AD5308ARUZ, U7 AD5308ARUZ

Commit message: Updade 1V ADC.brd enviada pra digikart
Parts:
- C1, C3: value 10nf -> 100nf
- C2, C4: value 10uf -> 4.7uf
- C5: value 10nf -> 1pf
- C6, C7, C8, C9: value 10nf -> 10pf
- R1, R3: value (none) -> 1.5k
- R2, R4: value (none) -> 3.3k
- R20, R21, R22, R48: value (none) -> 10k
Connections:
- net 1V: now also R19.2, R32.2, R46.2
- net GND: now also IC13A.INH, IC5A.INH, IC6A.INH, R48.2; no longer R19.2, R32.2, R46.2, U1.VREF_OUT, U4.VREF_OUT
- net N$103: now also U2.+INA; no longer R48.2
- net VCC: no longer IC13A.INH, IC5A.INH, IC6A.INH

Commit message: update
Parts:
- R17, R33, R49, R5, R50, R57: value (none) -> 10k
- R18, R51: value (none) -> 30K
- R19, R53: value (none) -> 3,3K
- R31, R45, R52, R55: value (none) -> 30k
- R32, R46, R54, R56: value (none) -> 3,3k
Changed lines of the file:
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@@
 <part name="R15" library="SparkFun" deviceset="RESISTOR" device="0603"/>
 <part name="R16" library="SparkFun" deviceset="RESISTOR" device="0603"/>
-<part name="R18" library="SparkFun" deviceset="RESISTOR" device="0603"/>
-<part name="R19" library="SparkFun" deviceset="RESISTOR" device="0603"/>
+<part name="R18" library="SparkFun" deviceset="RESISTOR" device="0603" value="30K"/>
+<part name="R19" library="SparkFun" deviceset="RESISTOR" device="0603" value="3,3K"/>
 <part name="U4" library="ADI-Phase-2" deviceset="ADV7173KSTZ" device=""/>
 <part name="SUPPLY30" library="supply2" deviceset="VDD" device=""/>
@@
 <part name="R29" library="SparkFun" deviceset="RESISTOR" device="0603"/>
 <part name="R30" library="SparkFun" deviceset="RESISTOR" device="0603"/>
-<part name="R31" library="SparkFun" deviceset="RESISTOR" device="0603"/>
-<part name="R32" library="SparkFun" deviceset="RESISTOR" device="0603"/>
+<part name="R31" library="SparkFun" deviceset="RESISTOR" device="0603" value="30k"/>
+<part name="R32" library="SparkFun" deviceset="RESISTOR" device="0603" value="3,3k"/>
 <part name="R34" library="SparkFun" deviceset="RESISTOR" device="0603"/>
 <part name="R35" library="SparkFun" deviceset="RESISTOR" device="0603"/>
@@
 <part name="R43" library="SparkFun" deviceset="RESISTOR" device="0603"/>
 <part name="R44" library="SparkFun" deviceset="RESISTOR" device="0603"/>
-<part name="R45" library="SparkFun" deviceset="RESISTOR" device="0603"/>
-<part name="R46" library="SparkFun" deviceset="RESISTOR" device="0603"/>
+<part name="R45" library="SparkFun" deviceset="RESISTOR" device="0603" value="30k"/>
+<part name="R46" library="SparkFun" deviceset="RESISTOR" device="0603" value="3,3k"/>
 <part name="SV1" library="con-lstb" deviceset="MA20-2" device=""/>
 <part name="U5" library="Analog Devices_By_element14_Batch_1" deviceset="AD5308ARUZ" device=""/>
@@
 <part name="SUPPLY20" library="supply2" deviceset="VDD" device=""/>
 <part name="R48" library="SparkFun" deviceset="RESISTOR" device="0603" value="10k"/>
-<part name="R5" library="SparkFun" deviceset="RESISTOR" device="0603"/>
-<part name="R49" library="SparkFun" deviceset="RESISTOR" device="0603"/>
-<part name="R51" library="SparkFun" deviceset="RESISTOR" device="0603"/>
-<part name="R53" library="SparkFun" deviceset="RESISTOR" device="0603"/>
-<part name="R17" library="SparkFun" deviceset="RESISTOR" device="0603"/>
-<part name="R50" library="SparkFun" deviceset="RESISTOR" device="0603"/>
-<part name="R52" library="SparkFun" deviceset="RESISTOR" device="0603"/>
-<part name="R54" library="SparkFun" deviceset="RESISTOR" device="0603"/>
-<part name="R55" library="SparkFun" deviceset="RESISTOR" device="0603"/>
-<part name="R56" library="SparkFun" deviceset="RESISTOR" device="0603"/>
-<part name="R57" library="SparkFun" deviceset="RESISTOR" device="0603"/>
-<part name="R33" library="SparkFun" deviceset="RESISTOR" device="0603"/>
+<part name="R5" library="SparkFun" deviceset="RESISTOR" device="0603" value="10k"/>
+<part name="R49" library="SparkFun" deviceset="RESISTOR" device="0603" value="10k"/>
+<part name="R51" library="SparkFun" deviceset="RESISTOR" device="0603" value="30K"/>
+<part name="R53" library="SparkFun" deviceset="RESISTOR" device="0603" value="3,3K"/>
+<part name="R17" library="SparkFun" deviceset="RESISTOR" device="0603" value="10k"/>
+<part name="R50" library="SparkFun" deviceset="RESISTOR" device="0603" value="10k"/>
+<part name="R52" library="SparkFun" deviceset="RESISTOR" device="0603" value="30k"/>
+<part name="R54" library="SparkFun" deviceset="RESISTOR" device="0603" value="3,3k"/>
+<part name="R55" library="SparkFun" deviceset="RESISTOR" device="0603" value="30k"/>
+<part name="R56" library="SparkFun" deviceset="RESISTOR" device="0603" value="3,3k"/>
+<part name="R57" library="SparkFun" deviceset="RESISTOR" device="0603" value="10k"/>
+<part name="R33" library="SparkFun" deviceset="RESISTOR" device="0603" value="10k"/>
 <part name="SUPPLY32" library="supply2" deviceset="GND" device=""/>
 <part name="SUPPLY21" library="supply2" deviceset="GND" device=""/>
@@
 <wire x1="373.38" y1="55.88" x2="551.18" y2="55.88" width="0.1524" layer="91"/>
 <pinref part="X2" gate="-3" pin="KL"/>
+<junction x="551.18" y="55.88"/>
+<junction x="368.3" y="55.88"/>
+<junction x="373.38" y="55.88"/>
 </segment>
 </net>

Commit message: atualização
FPGA - send ADC
C# - DFT
Placa - 2 grounds
Parts:
- removed U$1: POT100K_3362U, SparkFun:POT100K_3362U
- added C14, C15, C16, C17, C18, C19, C20, C21: 1uF, eagle-ltspice:CC0603
- added C22: (no value), capacitor-wima:C2,5-3
- added C23, C30: 10pf, eagle-ltspice:CC0603
- added C24: (no value), capacitor-wima:C10/6
- added R47, R58: 1.5k, SparkFun:RESISTOR0603
- C5: value 1pf -> 10pf
- R48: value 10k -> 1.5k
Connections:
- removed net N$8: U2.+IND
- new net DGND: C12.2, C13.2, C22.2, C24.2, C3.2, C30.2, C4.2, JP1.3, JP2.3, JP3.3, SV1.11, SV1.29, SV2.11, SV2.29, U1.GND, U1.GND_(, U1.GND_10, U1.GND_11, U1.GND_12, U1.GND_7, U1.GND_8, U1.GND_9, U1.S1, U4.GND, U4.GND_(, U4.GND_10, U4.GND_11, U4.GND_12, U4.GND_7, U4.GND_8, U4.GND_9
- new net N$109: R47.1, U3.RFB
- new net N$124: R1.2, R58.1, U2.OUTD
- new net VREF/INA: R19.2, R32.2, R46.2
- net +5V: now also C14.1, C16.1, C18.1, C20.1; no longer SV1.12, SV2.12
- net -5V: now also C15.1, C17.1, C19.1, C21.1
- net 1V: no longer R19.2, R32.2, R46.2
- net DAC_OUT: now also C5.1, R47.2, R48.2; no longer R1.2, U$1.A
- net DCLK: now also C30.1
- net GND: now also C14.2, C15.2, C16.2, C17.2, C18.2, C19.2, C20.2, C21.2, C22.1, C23.2, C24.1, U2.+INA, U2.+IND; no longer C12.2, C13.2, C3.2, C4.2, C5.2, JP1.3, JP2.3, JP3.3, R48.2, SV1.11, SV1.29, SV2.11, SV2.29, U1.GND, U1.GND_(, U1.GND_10, U1.GND_11, U1.GND_12, U1.GND_7, U1.GND_8, U1.GND_9, U3.RFB, U4.GND, U4.GND_(, U4.GND_10, U4.GND_11, U4.GND_12, U4.GND_7, U4.GND_8, U4.GND_9
- net N$103: now also C5.2, U2.-INA; no longer C5.1, U2.+INA
- net N$111: now also C23.1
- net N$3: now also R58.2, U2.-IND; no longer U$1.E, U$1.S, U2.-INA
- net S1: no longer U1.S1
- net S2: no longer U1.S2
- net VCC: now also X2-6.KL
- net VDD: now also U1.S2; no longer X2-6.KL
Other:
- moved on the sheet: C5, R48
