File: adc.brd (EAGLE design)
At the start: 96 x 95.3 mm, 86 parts, among them IC13 4051D, IC5 4051D, IC6 4051D, U1 ADV7173KSTZ, U2 AD5308ARUZ, U3 AD7927BRUZ, U4 ADV7173KSTZ, U5 AD5308ARUZ, U6 AD5308ARUZ, U7 AD5308ARUZ

Commit message: Updade 1V ADC.brd enviada pra digikart
Parts:
- C1, C3: value 10nf -> 100nf
- C2, C4: value 10uf -> 4.7uf
- C5: value 10nf -> 1pf
- C6, C7, C8, C9: value 10nf -> 10pf
- R1, R3: value (none) -> 1.5k
- R2, R4: value (none) -> 3.3k
- R20, R21, R22, R48: value (none) -> 10k
- moved R46 3.58 mm to (50.7, 62.8), turned to 270 degrees
- moved R32 1.75 mm to (54.4, 43.6)
- moved R31 0.99 mm to (52.3, 43.6)
- moved U$1 0.58 mm to (61.0, 23.5)
- moved R16 0.31 mm to (44.8, 26.9)
- moved R14 0.11 mm to (44.8, 29.3)
Connections:
- removed net +INA: U2.3
- net 1V: now also R19.2, R32.2, R46.2
- net GND: now also IC13.6, IC5.6, IC6.6, R48.2; no longer R19.2, R32.2, R46.2, U1.6, U4.6
- net N$103: now also U2.3; no longer R48.2
- net VCC: no longer IC13.6, IC5.6, IC6.6
Routing:
- net 1V: track 119.7 -> 251.8 mm, vias 0 -> 5
- net N$103: track 7.41 -> 30.1 mm
- net VCC: track 462.7 -> 454.5 mm, vias 11 -> 13
- net CH_C(ADC): track 65.0 -> 59.0 mm
- net GND: track 923.6 -> 918.7 mm
- net N$104: track 19.6 -> 16.3 mm
- net +5V: track 325.3 -> 327.9 mm
- net -5V: track 344.7 -> 342.2 mm
- net N$106: track 25.1 -> 24.0 mm, vias 0 -> 1
- net DAC_OUT: track 20.2 -> 19.2 mm
- net N$120: track 25.5 -> 24.8 mm
- net N$99: track 38.8 -> 38.3 mm
- net N$48: track 49.4 -> 49.9 mm
- net N$107: track 24.0 -> 24.3 mm, vias 0 -> 1

Commit message: update
Parts:
- R17, R33, R49, R5, R50, R57: value (none) -> 10k
- R18, R51: value (none) -> 30K
- R19, R53: value (none) -> 3,3K
- R31, R45, R52, R55: value (none) -> 30k
- R32, R46, R54, R56: value (none) -> 3,3k
Routing:
- net -5V: track 342.2 -> 337.3 mm

Commit message: Atualização
Parts:
- removed U$1: POT100K_3362U, SparkFun:3362U
- added C14, C15, C16, C17, C18, C19, C20, C21: 1uF, eagle-ltspice:C0603
- added C22: (no value), capacitor-wima:C2.5-3
- added C23, C30: 10pf, eagle-ltspice:C0603
- added C24: (no value), capacitor-wima:C10B6
- added R47, R58: 1.5k, SparkFun:0603
- C5: value 1pf -> 10pf
- R48: value 10k -> 1.5k
- moved R48 3.51 mm to (62.3, 25.7), turned to 180 degrees
- moved C5 2.20 mm to (61.8, 22.9), turned to 270 degrees
- moved R46 1.77 mm to (49.6, 61.4)
- moved R45 1.75 mm to (52.3, 62.9)
- moved R18 1.55 mm to (52.2, 19.7)
- moved R5 1.55 mm to (54.9, 20.4)
- moved R19 1.09 mm to (50.4, 23.0)
- moved R41 0.79 mm to (46.0, 62.3)
- moved R17 0.71 mm to (49.8, 37.7)
- moved R37 0.58 mm to (46.0, 64.6)
- moved R38 0.58 mm to (46.0, 67.1)
- moved R11 0.48 mm to (45.5, 19.5)
- moved R39 0.36 mm to (46.0, 69.4)
- moved R33 0.25 mm to (54.6, 65.6), turned to 90 degrees
Connections:
- removed net N$8: U2.14
- new net DGND: C12.2, C13.2, C22.2, C24.2, C3.2, C30.2, C4.2, JP1.3, JP2.3, JP3.3, SV1.11, SV1.29, SV2.11, SV2.29, U1.1, U1.12, U1.16, U1.27, U1.29, U1.32, U1.34, U1.45, U1.8, U4.1, U4.12, U4.16, U4.27, U4.29, U4.32, U4.34, U4.45
- new net N$109: R47.1, U3.20
- new net N$124: R1.2, R58.1, U2.16
- new net VEE: IC13.7, IC5.7, IC6.7
- new net VREF/INA: R19.2, R32.2, R46.2
- net +5V: now also C14.1, C16.1, C18.1, C20.1, IC13.16, IC5.16, IC6.16; no longer SV1.12, SV2.12
- net -5V: now also C15.1, C17.1, C19.1, C21.1
- net 1V: no longer R19.2, R32.2, R46.2
- net DAC_OUT: now also C5.1, R47.2, R48.2; no longer R1.2, U$1.P$3
- net DCLK: now also C30.1
- net GND: now also C14.2, C15.2, C16.2, C17.2, C18.2, C19.2, C20.2, C21.2, C22.1, C23.2, C24.1, U2.14, U2.3; no longer C12.2, C13.2, C3.2, C4.2, C5.2, JP1.3, JP2.3, JP3.3, R48.2, SV1.11, SV1.29, SV2.11, SV2.29, U1.1, U1.12, U1.16, U1.27, U1.29, U1.32, U1.34, U1.45, U3.20, U4.1, U4.12, U4.16, U4.27, U4.29, U4.32, U4.34, U4.45
- net N$103: now also C5.2, U2.2; no longer C5.1, U2.3
- net N$111: now also C23.1
- net N$3: now also R58.2, U2.15; no longer U$1.P$1, U$1.P$2, U2.2
- net S1: no longer U1.8
- net S2: no longer U1.9
- net VCC: now also X2.6; no longer IC13.16, IC5.16, IC6.16
- net VDD: now also U1.9; no longer X2.6
Routing:
- net DGND: track 0.00 -> 364.2 mm, vias 0 -> 8
- net GND: track 918.6 -> 750.8 mm, vias 17 -> 23
- net 1V: track 251.8 -> 119.9 mm, vias 5 -> 1
- net VREF/INA: track 0.00 -> 83.1 mm, vias 0 -> 5
- net VCC: track 454.5 -> 417.8 mm, vias 13 -> 10
- net DCLK: track 134.9 -> 101.5 mm
- net S1: track 59.1 -> 30.9 mm, vias 2 -> 1
- net +5V: track 327.9 -> 355.2 mm, vias 6 -> 12
- net S2: track 54.3 -> 33.8 mm
- net N$124: track 0.00 -> 19.3 mm, vias 0 -> 2
- net VDD: track 324.3 -> 337.1 mm, vias 3 -> 4
- net -5V: track 337.3 -> 348.7 mm
- net N$7: track 97.6 -> 105.9 mm
- net N$109: track 0.00 -> 6.89 mm
- net CH_C(ADC): track 59.0 -> 53.1 mm
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- added copper zone on layer 1, net DGND
- added copper zone on layer 16, net DGND
- added copper zone on layer 1, net GND
